File: hardware/DRO-Pico/DRO_Pico_V2.0.2.kicad_sch (KiCad schematic)
At the start: 41 parts, among them J1 Sensor1, J10 I/O, J11 Ser 1, J2 Sensor2, J3 Sensor3, J4 Sensor4, J5 Disp1, J6 Disp2, J7 Disp3, J8 Disp4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

Commit message: Add files via upload
Other:
- note added: "Display 4x 6-Digit LED TM1637"
Changed lines of the file:
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@@
+		)
+	)
+	(text "Display 4x 6-Digit LED TM1637"
+		(exclude_from_sim no)
+		(at 259.588 90.17 0)
+		(effects
+			(font
+				(size 1.27 1.27)
+			)
 		)
 	)
